File: PCB/syringe board 1.6.sch (EAGLE design)
At the start: 40 parts, among them IC1 A3967SLB, Q1 RESONATOR_CSTCE_V, U1 ATMEGA328P_TQFP, U2 PCA9306

Commit message: PCB update to 1.6
Parts:
- removed C5: 680pF, SparkFun-Capacitors:CAP0603-CAP
- removed JP1: (no value), SparkFun-Connectors:M06NO_SILK_FEMALE_PTH
- removed JP3: (no value), SparkFun:M041X04_NO_SILK
- removed JP6: (no value), SparkFun-Connectors:M031X03_NO_SILK
- added C1: 680pF, SparkFun-Capacitors:CAP0603-CAP
- added J1: RJ45, Andy-library:RJ45
- added J2: AVR_SPI_PROG_3X2NS, SparkFun-Connectors:AVR_SPI_PROG_3X2NS
- added J5: (no value), SparkFun-Connectors:CONN_021X02_NO_SILK
- added U$3: FIDUCIAL, adafruit:FIDUCIAL
- added U$5: OMRON_4PIN, Andy-library:OMRON_4PIN
- JP2: device SparkFun-Connectors:M05NO_SILK -> SparkFun-Connectors:M04NO_SILK_ALL_ROUND
- JP4: device SparkFun-Connectors:M04NO_SILK_ALL_ROUND -> SparkFun-Connectors:M05NO_SILK
- LED1: value (none) -> PWR
- R1: value .75 -> 3.3K; device SparkFun-Resistors:RESISTOR0805-RES -> SparkFun-Resistors:RESISTOR0603
- R16: value 3.3K -> 10K
- R17: value 6.8K -> 1K
- R2: value .75 -> 2.49K; device SparkFun-Resistors:RESISTOR0805-RES -> SparkFun-Resistors:RESISTOR0603
- R20: value 10K -> 1K
- R21: value 10K -> 200k
- R23: value 20k -> 1K
- R4: value 20K -> 20k
- R5: value 2.49K -> .75; device SparkFun-Resistors:RESISTOR0603 -> SparkFun-Resistors:RESISTOR0805-RES
- R6: value 200k -> .75; device SparkFun-Resistors:RESISTOR0603 -> SparkFun-Resistors:RESISTOR0805-RES
- R7: value 1K -> 10K
- R8: value 1K -> 20K
- R9: value 1K -> 6.8K
- U$1: value MICROSD_SOCKET -> FIDUCIAL; device Andy-library:MICROSD_SOCKET -> adafruit:FIDUCIAL
- U$2: value RJ45 -> FIDUCIAL; device Andy-library:RJ45 -> adafruit:FIDUCIAL
- renumbered PWR to LED1
Connections:
- removed net MISO: JP1.5, U$1.DATA_OUT, U1.PB4(MISO)
- removed net MOSI: JP1.4, U$1.DATA_IN, U1.PB3(MOSI/OC2)
- removed net N$13: U1.PB0(ICP)
- removed net SCK: JP1.6, U$1.CLK, U1.PB5(SCK)
- new net N$10: J2.3, U1.PB5(SCK)
- net 12VDC: now also J1.6; no longer U$2.6
- net 3VDC: now also J1.7, JP2.2, R17.1, R20.1; no longer JP4.2, JP6.1, R22.1, R9.1, U$1.VIN, U$2.7
- net 5VDC: now also J1.4, J2.2, R1.2, R13.2, R21.1, R22.1, R4.1, R7.2; no longer JP1.1, R10.2, R15.2, R16.2, R6.1, R7.1, R8.1, U$2.4
- net DIR_IN: now also R10.2; no longer R20.2
- net DISP_SCL: now also JP4.4, R20.2; no longer JP2.4, R22.2
- net DISP_SDA: now also JP4.5, R17.2; no longer JP2.5, R9.2
- net ENABLE: now also R15.2; no longer R13.2
- net GND: now also C1.2, J1.5, J2.6, JP2.4, R10.1, R15.1, R16.1, R6.1, R8.1, R9.1, U$5.GND1, U$5.GND2; no longer C5.2, JP1.2, JP4.4, JP6.2, R1.1, R13.1, R17.1, R20.1, R21.1, R4.1, U$1.G1, U$1.G2, U$1.G3, U$1.G4, U$1.GND, U$2.5
- net MCU_SCL: now also R22.2; no longer R7.2
- net MCU_SDA: now also R23.2; no longer R8.2
- net MS1: now also R12.1; no longer R14.1
- net MS2: now also R13.1; no longer R10.1
- net N$1: now also R5.2; no longer R1.2
- net N$11: now also J2.4, U1.PB3(MOSI/OC2); no longer U1.PB1(OC1A)
- net N$12: now also J1.3; no longer JP6.3, U$2.3
- net N$15: now also JP4.1; no longer JP2.1
- net N$16: now also JP4.2; no longer JP2.2
- net N$17: now also JP4.3; no longer JP2.3
- net N$20: now also J1.2; no longer U$2.2
- net N$21: now also J1.1; no longer U$2.1
- net N$3: now also R6.2; no longer R2.2
- net N$5: now also C1.1; no longer C4.1
- net N$6: now also R21.2; no longer R6.2
- net N$7: now also C4.1, R8.2; no longer C5.1, R4.2
- net N$8: now also R4.2; no longer R23.2
- net N$9: now also J2.1, U1.PB4(MISO); no longer U$1.CS, U1.PD7(AIN1)
- net OUT1A: now also U$5.P$2; no longer JP3.3
- net OUT1B: now also U$5.P$1; no longer JP3.4
- net OUT2A: now also U$5.P$4; no longer JP3.1
- net OUT2B: now also U$5.P$3; no longer JP3.2
- net PFD: now also R7.1, R9.2; no longer R12.1, R17.2
- net RESET: now also R14.1; no longer R15.1
- net RST: now also J2.5, JP2.1; no longer JP1.3, JP4.1
- net STEP_IN: now also R16.2; no longer R21.2
- net VREF: now also R1.1, R2.2; no longer R16.1, R5.2
Other:
- note removed: "Andy Lustig"
- note removed: "More info at: https://github.com/alustig3/Syringe-pump"
- moved on the sheet: C2, C3, C4, R1, R10, R12, R13, R14, R15, R16, R17, R2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
