File: pcb/syringe_board.kicad_sch (KiCad schematic)
At the start: 32 parts, among them J1 RJ45_pyControl, J2 PPTC161LFBN-RC, J3 PPTC121LFBN-RC, J4 Conn_02x03_Odd_Even, J5 Conn_01x04_Male, J6 Male header, J7 Female header, J8 Conn_01x04_Male, U1 AZ1117-3.3, U2 ATSAMD21G, U3 TMC2209, U4 AT24C01C-STUM, X1 feather_wing

Commit message: pcb v4.4
Parts:
- removed H1, H2: MountingHole, MountingHole:MountingHole_3.2mm_M3, symbol Mechanical:MountingHole
- removed H3: MountingHole, MountingHole:MountingHole_3.2mm_M3_DIN965_Pad, symbol Mechanical:MountingHole
- added H1, H2, H3: 9774010943R, asl_footprints:standoff_nut, symbol asl_symbols:Threaded_Standoff
- J1: value RJ45_pyControl -> 54602-908LF; footprint asl_footprints:RJ45_SMD -> asl_footprints:RJ45_THP_Vertical
- J2: value PPTC161LFBN-RC -> ESQ-116-12-T-S
- J3: value PPTC121LFBN-RC -> ESQ-112-12-T-S
- J4: renamed from J6; value Male header -> PH1RB-07-UA
- J5: renamed from J4; DNP (none) -> 1
- J6: renamed from J5; value Conn_01x04_Male -> Motor leads; DNP (none) -> 1
- J7: value Female header -> PPTC071LGBN-RC
- J8: value Conn_01x04_Male -> Limit switches; DNP (none) -> 1
- renumbered C2 to C1, C11 to C10, C3 to C2, C4 to C3, C5 to C4, C6 to C5, C7 to C6, C8 to C7, C9 to C8, C10 to C9, R3 to R1, R4 to R2, R2 to R3, R7 to R4, R6 to R5, R8 to R6
Connections:
- no-connect marks 0 -> 21
Other:
- note added: "Microcontroller and Feather Wing headers"
- note added: "Motor Driver"
- note added: "Motor and limit switch connections"
- note added: "Power and pyControl communication"
- moved on the sheet: C1, C10, C5, C6, C7, C8, C9, J2, J3, J4, J5, J6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

Commit message: pcb v1.5
- copper circular pad added back to mounting holes for durability
- added silkscreen hints on bottom side of motor lead/limit switch breakout
- added 3 right angle tactile switches
- changed to smaller 3.3v re3gulator
- one of limits was D10, now A1
Parts:
- removed C2: 22µF, Capacitor_SMD:C_1206_3216Metric, symbol Device:C
- removed C3: 10µF, Capacitor_SMD:C_1206_3216Metric, symbol Device:C
- removed U1: AZ1117-3.3, Package_TO_SOT_SMD:SOT-223, symbol Regulator_Linear:AZ1117-3.3
- added C2, C3: 2.2µF, Capacitor_SMD:C_0603_1608Metric, symbol Device:C_Small
- added S1, S2, S3: PTS645VH39-2, Button_Switch_THT:SW_Tactile_SPST_Angled_PTS645Vx39-2LFS, symbol asl_symbols:switch_momentary_2pin
- added U1: BU33SD2MG, Package_TO_SOT_SMD:SOT-23-5, symbol asl_symbols_new:BU33SD2MG
Connections:
- net +3V3: now also C2.1, U1.5 (Vout)
- net 5VDC: now also C3.1, U1.1 (Vin), U1.3 (STBY)
- net A1: now also J4.6 (Pin_6)
- net D10: now also S1.1; no longer J4.6 (Pin_6)
- net D12: now also S2.1
- net D13: now also S3.1
- net GND: now also C2.2, C3.2, S1.2, S2.2, S3.2, U1.2 (GND)

Commit message: up to date CAD
Parts:
- J1: footprint asl_footprints:RJ45_THP_Vertical -> asl_footprints:RJ45_THP
