File: ecad/controller.kicad_pcb (KiCad board)
At the start: 2 copper layers, 65 x 62 mm, 51 parts, among them J1 PPTC141LGBN-RC, J2 PEC14SBAN, J3 Conn_01x06_Socket, J4 Conn_01x06_Socket, J5 Conn_01x06_Socket, SW1 PEC11R-4220F-S0024, U1 TMC5041, U2 TMC5041

Commit message: change BOM to use 12-pin female header
Parts:
- J2: value PEC14SBAN -> PH1RB-14-UA
Changed lines of the file:
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@@
 			)
 		)
-		(property "Datasheet" ""
+		(property "Datasheet" "~"
 			(at 0 0 0)
 			(unlocked yes)
@@
 		(sheetname "/")
 		(sheetfile "controller.kicad_sch")
-		(attr through_hole)
+		(attr through_hole exclude_from_bom)
 		(fp_line
 			(start 1.33 -1.27)
@@
 			)
 		)
-		(property "Datasheet" ""
+		(property "Datasheet" "~"
 			(at 0 0 0)
 			(unlocked yes)
@@
 		(sheetname "/")
 		(sheetfile "controller.kicad_sch")
-		(attr through_hole)
+		(attr through_hole exclude_from_bom)
 		(fp_line
 			(start 1.33 -1.27)
@@
 			)
 		)
-		(property "Value" "PEC14SBAN"
+		(property "Value" "PH1RB-14-UA"
 			(at 4.385 -35.29 0)
 			(layer "B.Fab")
@@
 			)
 		)
-		(property "Datasheet" "https://www.digikey.com/en/products/detail/sullins-connector-solutions/PEC14SBAN/860103?s=N4IgTCBcDaIM4EYlgKYFoEBYQF0C+QA"
+		(property "Datasheet" "https://www.digikey.com/en/products/detail/adam-tech/PH1RB-14-UA/9831063?s=N4IgTCBcDa4AwFYDsBaACgCQIwCUBCKWALCgKoCCKAcgCIgC6AvkA"
 			(at 0 0 180)
 			(unlocked yes)
@@
 			)
 		)
-		(property "Datasheet" ""
+		(property "Datasheet" "~"
 			(at 0 0 0)
 			(unlocked yes)
@@
 		(sheetname "/")
 		(sheetfile "controller.kicad_sch")
-		(attr through_hole)
+		(attr through_hole exclude_from_bom)
 		(fp_line
 			(start 1.33 -1.27)
